File: TJA1441.kicad_sch (KiCad schematic)
At the start: 5 parts

Commit message: CANの終端抵抗を削除、シルクスクリーンを調整
Parts:
- removed JP1: TR, Connector_PinHeader_2.54mm:PinHeader_1x02_P2.54mm_Vertical, symbol Jumper:Jumper_2_Small_Open
- renumbered R6 to R7
Connections:
- net FDCAN_H: now also R7.1
Other:
- moved on the sheet: R7
Changed lines of the file:
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@@
 	(wire
 		(pts
-			(xy 120.65 59.69) (xy 120.65 62.23)
+			(xy 120.65 59.69) (xy 120.65 64.77)
 		)
 		(stroke
@@
 	(wire
 		(pts
-			(xy 120.65 72.39) (xy 120.65 74.93)
+			(xy 120.65 69.85) (xy 120.65 74.93)
 		)
 		(stroke
@@
 		(on_board yes)
 		(dnp no)
-		(property "Reference" "#PWR038"
+		(property "Reference" "#PWR040"
 			(at 78.74 77.47 0)
 			(effects
@@
 			(project "DRC-CCTL2026"
 				(path "/5b9f915a-dea8-4ee6-a342-61437447bbca/0dbeca16-7879-4708-bbfc-c767bc55099f"
-					(reference "#PWR038")
+					(reference "#PWR040")
 					(unit 1)
 				)
 				(path "/5b9f915a-dea8-4ee6-a342-61437447bbca/8961d3ed-2b54-4595-a187-2d9f43ade7c1"
-					(reference "#PWR043")
+					(reference "#PWR045")
 					(unit 1)
 				)
 				(path "/5b9f915a-dea8-4ee6-a342-61437447bbca/ca8f340b-c206-4785-b43a-605b2d347bc5"
-					(reference "#PWR048")
-					(unit 1)
-				)
-			)
-		)
-	)
-	(symbol
-		(lib_id "Jumper:Jumper_2_Small_Open")
-		(at 120.65 64.77 270)
-		(unit 1)
-		(exclude_from_sim no)
-		(in_bom yes)
-		(on_board yes)
-		(dnp no)
-		(fields_autoplaced yes)
-		(property "Reference" "JP1"
-			(at 123.19 63.4999 90)
-			(effects
-				(font
-					(size 1.27 1.27)
-				)
-				(justify left)
-			)
-		)
-		(property "Value" "TR"
-			(at 123.19 66.0399 90)
-			(effects
-				(font
-					(size 1.27 1.27)
-				)
-				(justify left)
-			)
-		)
-		(property "Footprint" "Connector_PinHeader_2.54mm:PinHeader_1x02_P2.54mm_Vertical"
-			(at 120.65 64.77 0)
-			(effects
-				(font
-					(size 1.27 1.27)
-				)
-				(hide yes)
-			)
-		)
-		(property "Datasheet" "~"
-			(at 120.65 64.77 0)
-			(effects
-				(font
-					(size 1.27 1.27)
-				)
-				(hide yes)
-			)
-		)
-		(property "Description" "Jumper, 2-pole, small symbol, open"
-			(at 120.65 64.77 0)
-			(effects
-				(font
-					(size 1.27 1.27)
-				)
-				(hide yes)
-			)
-		)
-		(pin "1"
-		)
-		(pin "2"
-		)
-		(instances
-			(project "DRC-CCTL2026"
-				(path "/5b9f915a-dea8-4ee6-a342-61437447bbca/0dbeca16-7879-4708-bbfc-c767bc55099f"
-					(reference "JP1")
-					(unit 1)
-				)
-				(path "/5b9f915a-dea8-4ee6-a342-61437447bbca/8961d3ed-2b54-4595-a187-2d9f43ade7c1"
-					(reference "JP2")
-					(unit 1)
-				)
-				(path "/5b9f915a-dea8-4ee6-a342-61437447bbca/ca8f340b-c206-4785-b43a-605b2d347bc5"
-					(reference "JP3")
+					(reference "#PWR050")
 					(unit 1)
 				)
@@
 		(on_board yes)
 		(dnp no)
-		(property "Reference" "#PWR042"
+		(property "Reference" "#PWR044"
 			(at 104.14 88.9 0)
 			(effects
@@
 			(project "DRC-CCTL2026"
 				(path "/5b9f915a-dea8-4ee6-a342-61437447bbca/0dbeca16-7879-4708-bbfc-c767bc55099f"
-					(reference "#PWR042")
+					(reference "#PWR044")
 					(unit 1)
 				)
 				(path "/5b9f915a-dea8-4ee6-a342-61437447bbca/8961d3ed-2b54-4595-a187-2d9f43ade7c1"
-					(reference "#PWR047")
+					(reference "#PWR049")
 					(unit 1)
 				)
 				(path "/5b9f915a-dea8-4ee6-a342-61437447bbca/ca8f340b-c206-4785-b43a-605b2d347bc5"
-					(reference "#PWR052")
+					(reference "#PWR054")
 					(unit 1)
 				)
@@
 	(symbol
 		(lib_id "lib:R_Small")
-		(at 120.65 69.85 0)
+		(at 120.65 67.31 0)
 		(unit 1)
 		(exclude_from_sim no)
@@
 		(on_board yes)
 		(dnp no)
-		(property "Reference" "R6"
+		(property "Reference" "R7"
+			(at 121.92 66.04 0)
+			(effects
+				(font
+					(size 1.27 1.27)
+				)
+				(justify left)
+			)
+		)
+		(property "Value" "120"
 			(at 121.92 68.58 0)
 			(effects
@@
 			)
 		)
-		(property "Value" "120"
-			(at 121.92 71.12 0)
-			(effects
-				(font
-					(size 1.27 1.27)
-				)
-				(justify left)
-			)
-		)
 		(property "Footprint" "Resistor_SMD:R_0603_1608Metric_Pad0.98x0.95mm_HandSolder"
-			(at 120.65 69.85 0)
+			(at 120.65 67.31 0)
 			(effects
 				(font
@@
 		)
 		(property "Datasheet" "~"
-			(at 120.65 69.85 0)
+			(at 120.65 67.31 0)
 			(effects
 				(font
@@
 		)
 		(property "Description" "Resistor, small symbol"
-			(at 120.65 69.85 0)
+			(at 120.65 67.31 0)
 			(effects
 				(font
@@
 			(project "DRC-CCTL2026"
 				(path "/5b9f915a-dea8-4ee6-a342-61437447bbca/0dbeca16-7879-4708-bbfc-c767bc55099f"
-					(reference "R6")
+					(reference "R7")
 					(unit 1)
 				)
 				(path "/5b9f915a-dea8-4ee6-a342-61437447bbca/8961d3ed-2b54-4595-a187-2d9f43ade7c1"
-					(reference "R7")
+					(reference "R8")
 					(unit 1)
 				)
 				(path "/5b9f915a-dea8-4ee6-a342-61437447bbca/ca8f340b-c206-4785-b43a-605b2d347bc5"
-					(reference "R8")
+					(reference "R9")
 					(unit 1)
 				)
@@
 		(on_board yes)
 		(dnp no)
-		(property "Reference" "#PWR039"
+		(property "Reference" "#PWR041"
 			(at 88.9 72.39 0)
 			(effects
@@
 			(project "DRC-CCTL2026"
 				(path "/5b9f915a-dea8-4ee6-a342-61437447bbca/0dbeca16-7879-4708-bbfc-c767bc55099f"
-					(reference "#PWR039")
+					(reference "#PWR041")
 					(unit 1)
 				)
 				(path "/5b9f915a-dea8-4ee6-a342-61437447bbca/8961d3ed-2b54-4595-a187-2d9f43ade7c1"
-					(reference "#PWR044")
+					(reference "#PWR046")
 					(unit 1)
 				)
 				(path "/5b9f915a-dea8-4ee6-a342-61437447bbca/ca8f340b-c206-4785-b43a-605b2d347bc5"
-					(reference "#PWR049")
+					(reference "#PWR051")
 					(unit 1)
 				)
@@
 		(on_board yes)
 		(dnp no)
-		(property "Reference" "#PWR040"
+		(property "Reference" "#PWR042"
 			(at 96.52 60.96 0)
 			(effects
@@
 			(project "DRC-CCTL2026"
 				(path "/5b9f915a-dea8-4ee6-a342-61437447bbca/0dbeca16-7879-4708-bbfc-c767bc55099f"
-					(reference "#PWR040")
+					(reference "#PWR042")
 					(unit 1)
 				)
 				(path "/5b9f915a-dea8-4ee6-a342-61437447bbca/8961d3ed-2b54-4595-a187-2d9f43ade7c1"
-					(reference "#PWR045")
+					(reference "#PWR047")
 					(unit 1)
 				)
 				(path "/5b9f915a-dea8-4ee6-a342-61437447bbca/ca8f340b-c206-4785-b43a-605b2d347bc5"
-					(reference "#PWR050")
+					(reference "#PWR052")
 					(unit 1)
 				)
@@
 		(on_board yes)
 		(dnp no)
-		(property "Reference" "#PWR041"
+		(property "Reference" "#PWR043"
 			(at 104.14 55.88 0)
 			(effects
@@
 			(project "DRC-CCTL2026"
 				(path "/5b9f915a-dea8-4ee6-a342-61437447bbca/0dbeca16-7879-4708-bbfc-c767bc55099f"
-					(reference "#PWR041")
+					(reference "#PWR043")
 					(unit 1)
 				)
 				(path "/5b9f915a-dea8-4ee6-a342-61437447bbca/8961d3ed-2b54-4595-a187-2d9f43ade7c1"
-					(reference "#PWR046")
+					(reference "#PWR048")
 					(unit 1)
 				)
 				(path "/5b9f915a-dea8-4ee6-a342-61437447bbca/ca8f340b-c206-4785-b43a-605b2d347bc5"
-					(reference "#PWR051")
-					(unit 1)
-				)
+					(reference "#PWR053")
+					(unit 1)
+				)

Commit message: v0.2.0
Parts:
- FDCAN1: footprint footprints:SOIC127P600X175-8N -> lib:SO8_SOT96-1_NXP
- renumbered C17 to C3, C18 to C4
Changed lines of the file:
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@@
 		(on_board yes)
 		(dnp no)
-		(property "Reference" "#PWR040"
+		(property "Reference" "#PWR020"
 			(at 78.74 77.47 0)
 			(effects
@@
 			(project "DRC-CCTL2026"
 				(path "/5b9f915a-dea8-4ee6-a342-61437447bbca/0dbeca16-7879-4708-bbfc-c767bc55099f"
-					(reference "#PWR040")
-					(unit 1)
-				)
-				(path "/5b9f915a-dea8-4ee6-a342-61437447bbca/8961d3ed-2b54-4595-a187-2d9f43ade7c1"
-					(reference "#PWR045")
-					(unit 1)
-				)
-				(path "/5b9f915a-dea8-4ee6-a342-61437447bbca/ca8f340b-c206-4785-b43a-605b2d347bc5"
-					(reference "#PWR050")
+					(reference "#PWR020")
+					(unit 1)
+				)
+				(path "/5b9f915a-dea8-4ee6-a342-61437447bbca/8961d3ed-2b54-4595-a187-2d9f43ade7c1"
+					(reference "#PWR025")
+					(unit 1)
+				)
+				(path "/5b9f915a-dea8-4ee6-a342-61437447bbca/ca8f340b-c206-4785-b43a-605b2d347bc5"
+					(reference "#PWR030")
 					(unit 1)
 				)
@@
 		(on_board yes)
 		(dnp no)
-		(property "Reference" "C17"
+		(property "Reference" "C3"
 			(at 84.328 68.834 90)
 			(effects
@@
 			(project "DRC-CCTL2026"
 				(path "/5b9f915a-dea8-4ee6-a342-61437447bbca/0dbeca16-7879-4708-bbfc-c767bc55099f"
-					(reference "C17")
-					(unit 1)
-				)
-				(path "/5b9f915a-dea8-4ee6-a342-61437447bbca/8961d3ed-2b54-4595-a187-2d9f43ade7c1"
-					(reference "C19")
-					(unit 1)
-				)
-				(path "/5b9f915a-dea8-4ee6-a342-61437447bbca/ca8f340b-c206-4785-b43a-605b2d347bc5"
-					(reference "C21")
+					(reference "C3")
+					(unit 1)
+				)
+				(path "/5b9f915a-dea8-4ee6-a342-61437447bbca/8961d3ed-2b54-4595-a187-2d9f43ade7c1"
+					(reference "C5")
+					(unit 1)
+				)
+				(path "/5b9f915a-dea8-4ee6-a342-61437447bbca/ca8f340b-c206-4785-b43a-605b2d347bc5"
+					(reference "C7")
 					(unit 1)
 				)
@@
 		(on_board yes)
 		(dnp no)
-		(property "Reference" "#PWR044"
+		(property "Reference" "#PWR024"
 			(at 104.14 88.9 0)
 			(effects
@@
 			(project "DRC-CCTL2026"
 				(path "/5b9f915a-dea8-4ee6-a342-61437447bbca/0dbeca16-7879-4708-bbfc-c767bc55099f"
-					(reference "#PWR044")
-					(unit 1)
-				)
-				(path "/5b9f915a-dea8-4ee6-a342-61437447bbca/8961d3ed-2b54-4595-a187-2d9f43ade7c1"
-					(reference "#PWR049")
-					(unit 1)
-				)
-				(path "/5b9f915a-dea8-4ee6-a342-61437447bbca/ca8f340b-c206-4785-b43a-605b2d347bc5"
-					(reference "#PWR054")
+					(reference "#PWR024")
+					(unit 1)
+				)
+				(path "/5b9f915a-dea8-4ee6-a342-61437447bbca/8961d3ed-2b54-4595-a187-2d9f43ade7c1"
+					(reference "#PWR029")
+					(unit 1)
+				)
+				(path "/5b9f915a-dea8-4ee6-a342-61437447bbca/ca8f340b-c206-4785-b43a-605b2d347bc5"
+					(reference "#PWR034")
 					(unit 1)
 				)
@@
 		(on_board yes)
 		(dnp no)
-		(property "Reference" "C18"
+		(property "Reference" "C4"
 			(at 100.33 49.022 90)
 			(effects
@@
 			(project "DRC-CCTL2026"
 				(path "/5b9f915a-dea8-4ee6-a342-61437447bbca/0dbeca16-7879-4708-bbfc-c767bc55099f"
-					(reference "C18")
-					(unit 1)
-				)
-				(path "/5b9f915a-dea8-4ee6-a342-61437447bbca/8961d3ed-2b54-4595-a187-2d9f43ade7c1"
-					(reference "C20")
-					(unit 1)
-				)
-				(path "/5b9f915a-dea8-4ee6-a342-61437447bbca/ca8f340b-c206-4785-b43a-605b2d347bc5"
-					(reference "C22")
+					(reference "C4")
+					(unit 1)
+				)
+				(path "/5b9f915a-dea8-4ee6-a342-61437447bbca/8961d3ed-2b54-4595-a187-2d9f43ade7c1"
+					(reference "C6")
+					(unit 1)
+				)
+				(path "/5b9f915a-dea8-4ee6-a342-61437447bbca/ca8f340b-c206-4785-b43a-605b2d347bc5"
+					(reference "C8")
 					(unit 1)
 				)
@@
 		(on_board yes)
 		(dnp no)
-		(property "Reference" "#PWR041"
+		(property "Reference" "#PWR021"
 			(at 88.9 72.39 0)
 			(effects
@@
 			(project "DRC-CCTL2026"
 				(path "/5b9f915a-dea8-4ee6-a342-61437447bbca/0dbeca16-7879-4708-bbfc-c767bc55099f"
-					(reference "#PWR041")
-					(unit 1)
-				)
-				(path "/5b9f915a-dea8-4ee6-a342-61437447bbca/8961d3ed-2b54-4595-a187-2d9f43ade7c1"
-					(reference "#PWR046")
-					(unit 1)
-				)
-				(path "/5b9f915a-dea8-4ee6-a342-61437447bbca/ca8f340b-c206-4785-b43a-605b2d347bc5"
-					(reference "#PWR051")
+					(reference "#PWR021")
+					(unit 1)
+				)
+				(path "/5b9f915a-dea8-4ee6-a342-61437447bbca/8961d3ed-2b54-4595-a187-2d9f43ade7c1"
+					(reference "#PWR026")
+					(unit 1)
+				)
+				(path "/5b9f915a-dea8-4ee6-a342-61437447bbca/ca8f340b-c206-4785-b43a-605b2d347bc5"
+					(reference "#PWR031")
 					(unit 1)
 				)
@@
 		(on_board yes)
 		(dnp no)
-		(property "Reference" "#PWR042"
+		(property "Reference" "#PWR022"
 			(at 96.52 60.96 0)
 			(effects
@@
 			(project "DRC-CCTL2026"
 				(path "/5b9f915a-dea8-4ee6-a342-61437447bbca/0dbeca16-7879-4708-bbfc-c767bc55099f"
-					(reference "#PWR042")
-					(unit 1)
-				)
-				(path "/5b9f915a-dea8-4ee6-a342-61437447bbca/8961d3ed-2b54-4595-a187-2d9f43ade7c1"
-					(reference "#PWR047")
-					(unit 1)
-				)
-				(path "/5b9f915a-dea8-4ee6-a342-61437447bbca/ca8f340b-c206-4785-b43a-605b2d347bc5"
-					(reference "#PWR052")
+					(reference "#PWR022")
+					(unit 1)
+				)
+				(path "/5b9f915a-dea8-4ee6-a342-61437447bbca/8961d3ed-2b54-4595-a187-2d9f43ade7c1"
+					(reference "#PWR027")
+					(unit 1)
+				)
+				(path "/5b9f915a-dea8-4ee6-a342-61437447bbca/ca8f340b-c206-4785-b43a-605b2d347bc5"
+					(reference "#PWR032")
 					(unit 1)
 				)
@@
 		(on_board yes)
 		(dnp no)
-		(property "Reference" "#PWR043"
+		(property "Reference" "#PWR023"
 			(at 104.14 55.88 0)
 			(effects
@@
 			(project "DRC-CCTL2026"
 				(path "/5b9f915a-dea8-4ee6-a342-61437447bbca/0dbeca16-7879-4708-bbfc-c767bc55099f"
-					(reference "#PWR043")
-					(unit 1)
-				)
-				(path "/5b9f915a-dea8-4ee6-a342-61437447bbca/8961d3ed-2b54-4595-a187-2d9f43ade7c1"
-					(reference "#PWR048")
-					(unit 1)
-				)
-				(path "/5b9f915a-dea8-4ee6-a342-61437447bbca/ca8f340b-c206-4785-b43a-605b2d347bc5"
-					(reference "#PWR053")
+					(reference "#PWR023")
+					(unit 1)
+				)
+				(path "/5b9f915a-dea8-4ee6-a342-61437447bbca/8961d3ed-2b54-4595-a187-2d9f43ade7c1"
+					(reference "#PWR028")
+					(unit 1)
+				)
+				(path "/5b9f915a-dea8-4ee6-a342-61437447bbca/ca8f340b-c206-4785-b43a-605b2d347bc5"
+					(reference "#PWR033")
 					(unit 1)
 				)
@@
 			)
 		)
-		(property "Footprint" "footprints:SOIC127P600X175-8N"
+		(property "Footprint" "lib:SO8_SOT96-1_NXP"
 			(at 114.3 157.15 0)
 			(effects
