File: STM32G474RET.kicad_sch (KiCad schematic)
At the start: 13 parts, among them SW3 SW_Push, U4 STM32G474RETx

Commit message: v0.2.1, USB CDC に対応
Connections:
- net BZ_TIM15_CH2: now reaches U4.37 (PB15)
- net USB_CDC_DP: now reaches U4.46 (PA12)
- net BZ_TIM1_CH4 renamed USB_CDC_DM
- net UART_USB1_RX: no longer names the net of U4.55 (PD2)
- net UART_USB1_TX: no longer names the net of U4.54 (PC12)
- net USART_USB2_RX renamed USART_USB_RX
- net USART_USB2_TX renamed USART_USB_TX
Changed lines of the file:
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@@
-	)
-	(no_connect
-		(at 168.91 152.4)
 	)
 	(no_connect
@@
 	)
 	(no_connect
+		(at 133.35 88.9)
+	)
+	(no_connect
 		(at 133.35 127)
 	)
@@
 	)
 	(no_connect
+		(at 133.35 124.46)
+	)
+	(no_connect
 		(at 168.91 71.12)
 	)
-	(no_connect
-		(at 168.91 101.6)
-	)
 	(wire
 		(pts
@@
 	(wire
 		(pts
-			(xy 121.92 88.9) (xy 133.35 88.9)
-		)
-		(stroke
-			(width 0)
-			(type default)
-		)
-	)
-	(wire
-		(pts
 			(xy 105.41 49.53) (xy 105.41 55.88)
 		)
@@
 	(wire
 		(pts
+			(xy 168.91 99.06) (xy 180.34 99.06)
+		)
+		(stroke
+			(width 0)
+			(type default)
+		)
+	)
+	(wire
+		(pts
+			(xy 168.91 101.6) (xy 180.34 101.6)
+		)
+		(stroke
+			(width 0)
+			(type default)
+		)
+	)
+	(wire
+		(pts
 			(xy 168.91 137.16) (xy 180.34 137.16)
 		)
@@
 	(wire
 		(pts
-			(xy 168.91 99.06) (xy 180.34 99.06)
+			(xy 168.91 152.4) (xy 180.34 152.4)
 		)
 		(stroke
@@
 		(pts
 			(xy 90.17 49.53) (xy 90.17 53.34)
-		)
-		(stroke
-			(width 0)
-			(type default)
-		)
-	)
-	(wire
-		(pts
-			(xy 121.92 124.46) (xy 133.35 124.46)
 		)
 		(stroke
@@
 		)
 	)
-	(hierarchical_label "USART_USB2_TX"
+	(hierarchical_label "USART_USB_TX"
 		(shape input)
 		(at 121.92 119.38 180)
@@
 		(shape input)
 		(at 121.92 99.06 180)
-		(effects
-			(font
-				(size 1.27 1.27)
-			)
-			(justify right)
-		)
-	)
-	(hierarchical_label "UART_USB1_RX"
-		(shape input)
-		(at 121.92 88.9 180)
 		(effects
 			(font
@@
 		)
 	)
+	(hierarchical_label "USB_CDC_DP"
+		(shape input)
+		(at 180.34 101.6 0)
+		(effects
+			(font
+				(size 1.27 1.27)
+			)
+			(justify left)
+		)
+	)
 	(hierarchical_label "LCD_SDA"
 		(shape input)
@@
 		)
 	)
-	(hierarchical_label "USART_USB2_RX"
+	(hierarchical_label "USART_USB_RX"
 		(shape input)
 		(at 121.92 121.92 180)
@@
 		)
 	)
-	(hierarchical_label "UART_USB1_TX"
-		(shape input)
-		(at 121.92 124.46 180)
-		(effects
-			(font
-				(size 1.27 1.27)
-			)
-			(justify right)
-		)
-	)
 	(hierarchical_label "FDCAN2_RX"
 		(shape input)
@@
 		(shape input)
 		(at 180.34 116.84 0)
+		(effects
+			(font
+				(size 1.27 1.27)
+			)
+			(justify left)
+		)
+	)
+	(hierarchical_label "USB_CDC_DM"
+		(shape input)
+		(at 180.34 99.06 0)
 		(effects
 			(font
@@
 		)
 	)
-	(hierarchical_label "BZ_TIM1_CH4"
-		(shape input)
-		(at 180.34 99.06 0)
-		(effects
-			(font
+	(hierarchical_label "BZ_TIM15_CH2"
+		(shape input)
+		(at 180.34 152.4 0)
+		(effects
+			(font
