File: DRC-CCTL2026.kicad_pcb (KiCad board)
At the start: 2 copper layers, 80 x 60 mm, 81 parts, among them J1 STLINK, J10 USB_C, J12 USB_C, J2 FDCAN1, J3 FDCAN2, J4 FDCAN3, J5 SW1, J6 SW2, J7 SW3, J8 I2C1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

Commit message: バージョン表記を修正・JLCPCBに書き出し
Other:
- board text added: "DRC-CCTL2026 v0.2.1"
- board text removed: "DRC-CCTL2026 v0.2.0"
Changed lines of the file:
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@@
 		)
 	)
-	(gr_text "DRC-CCTL2026 v0.2.0"
+	(gr_text "DRC-CCTL2026 v0.2.1"
 		(at 151.91 116.665 0)
 		(layer "B.SilkS")
@@
 			(justify left bottom mirror)
 		)
-		(render_cache "DRC-CCTL2026 v0.2.0" 0
+		(render_cache "DRC-CCTL2026 v0.2.1" 0
 			(polygon
 				(pts
@@
 			(polygon
 				(pts
-					(xy 123.143013 114.304566) (xy 123.205207 114.31589) (xy 123.318745 114.359642) (xy 123.420413 114.431513)
-					(xy 123.511374 114.533581) (xy 123.59085 114.669393) (xy 123.656081 114.842421) (xy 123.702667 115.054103)
-					(xy 123.725327 115.301552) (xy 123.726695 115.382466) (xy 123.722647 115.536682) (xy 123.709941 115.684783)
-					(xy 123.691237 115.807016) (xy 123.664824 115.922145) (xy 123.63486 116.016402) (xy 123.598163 116.103512)
-					(xy 123.559493 116.174468) (xy 123.514919 116.238574) (xy 123.468971 116.290525) (xy 123.417709 116.335918)
-					(xy 123.364644 116.372149) (xy 123.30657 116.401901) (xy 123.245352 116.42423) (xy 123.179125 116.439835)
-					(xy 123.05747 116.450052) (xy 122.990221 116.446202) (xy 122.926958 116.434882) (xy 122.812426 116.391349)
-					(xy 122.710836 116.320178) (xy 122.62065 116.219428) (xy 122.542262 116.08544) (xy 122.478048 115.914269)
-					(xy 122.432065 115.703538) (xy 122.409398 115.454781) (xy 122.408052 115.376849) (xy 122.746671 115.376849)
-					(xy 122.750741 115.534419) (xy 122.763597 115.68441) (xy 122.78183 115.800884) (xy 122.807475 115.906215)
-					(xy 122.834466 115.982482) (xy 122.867152 116.047983) (xy 122.898697 116.092956) (xy 122.934528 116.128736)
-					(xy 122.968861 116.151499) (xy 123.006602 116.166342) (xy 123.05747 116.172958) (xy 123.103077 116.16912)
-					(xy 123.144593 116.157883) (xy 123.215649 116.115224) (xy 123.275759 116.04323) (xy 123.326321 115.934169)
-					(xy 123.365404 115.776589) (xy 123.388897 115.556925) (xy 123.393426 115.379658) (xy 123.389434 115.226958)
-					(xy 123.377124 115.082496) (xy 123.359055 114.965078) (xy 123.333842 114.858869) (xy 123.306704 114.779509)
-					(xy 123.274012 114.711154) (xy 123.242191 114.663349) (xy 123.206203 114.625043) (xy 123.171854 114.600325)
-					(xy 123.134261 114.583731) (xy 123.077131 114.575122) (xy 123.031531 114.578965) (xy 122.990106 114.590234)
-					(xy 122.919772 114.632864) (xy 122.860691 114.704785) (xy 122.811283 114.814116) (xy 122.773341 114.973307)
-					(xy 122.7508 115.198374) (xy 122.746671 115.376849) (xy 122.408052 115.376849) (xy 122.407906 115.368422)
-					(xy 122.411896 115.223888) (xy 122.424191 115.08429) (xy 122.44292 114.963335) (xy 122.469239 114.848867)
-					(xy 122.499653 114.752525) (xy 122.53675 114.663189) (xy 122.576097 114.589424) (xy 122.621272 114.522633)
-					(xy 122.667739 114.468295) (xy 122.719364 114.420738) (xy 122.772342 114.382871) (xy 122.830063 114.351696)
-					(xy 122.89014 114.328385) (xy 122.954818 114.311945) (xy 123.077131 114.300715)
-				)
-			)
+					(xy 122.629068 116.410973) (xy 122.608558 116.407062) (xy 122.594178 116.395313) (xy 122.587058 116.369085)
+					(xy 122.587058 116.223394) (xy 122.591607 116.192269) (xy 122.602411 116.181303) (xy 122.62345 116.175889)
+					(xy 122.766441 116.159312) (xy 122.805588 116.144707) (xy 122.829037 116.122524) (xy 122.84412 116.071923)
+					(xy 122.847543 116.024459) (xy 122.853742 115.856894) (xy 122.855847 115.769469) (xy 122.851401 115.112098)
+					(xy 122.835906 114.594026) (xy 122.822264 114.399023) (xy 122.819455 114.354204) (xy 122.823469 114.32523)
+					(xy 122.835935 114.310458) (xy 122.855847 114.306577) (xy 122.883935 114.309385) (xy 123.044476 114.333444)
+					(xy 123.181034 114.345439) (xy 123.30672 114.348586) (xy 123.359842 114.348586) (xy 123.37636 114.352711)
+					(xy 123.388858 114.365954) (xy 123.393426 114.387787) (xy 123.394784 114.465813) (xy 123.396235 114.550209)
+					(xy 123.390632 114.587609) (xy 123.379697 114.595409) (xy 123.359842 114.597714) (xy 123.209114 114.603158)
+					(xy 123.177264 114.611693) (xy 123.163875 114.625638) (xy 123.161029 114.648272) (xy 123.155533 114.998639)
+					(xy 123.167362 115.725455) (xy 123.18069 116.027267) (xy 123.191203 116.103558) (xy 123.210709 116.139482)
+					(xy 123.253475 116.156228) (xy 123.346218 116.169067) (xy 123.429818 116.17308) (xy 123.444984 116.181318)
+					(xy 123.457987 116.199581) (xy 123.460715 116.21509) (xy 123.458762 116.314938) (xy 123.457906 116.352233)
+					(xy 123.453892 116.384195) (xy 123.441426 116.40442) (xy 123.421514 116.410973) (xy 123.415896 116.410973)
+					(xy 123.01546 116.402669) (xy 122.634685 116.410973)
+				)
+			)
